Commit message: 基于ManiSkill，扩充XArm6机械臂的任务至与Panda一致，调整各任务的解决方案使之更合理，并全部添加腕部相机与新的第三视角相机支持
支持robot_uid：panda_wristcam、panda_stick_wristcam、xarm6_robotiq_wristcam、xarm6_stick_wristcam
支持任务："PickCube-v1", "PullCube-v1", "PushCube-v1", "StackCube-v1", "PullCubeTool-v1", "PlaceSphere-v1", "LiftPegUpright-v1", "PegInsertionSide-v1", "DrawTriangle-v1", "DrawSVG-v1"

File: mani_skill/assets/robots/panda/panda_stick.urdf (robot description, URDF)
Before this commit: robot panda, 11 links, 10 joints
Links:
- added link camera_base_link
- added link camera_link, mass 0.564; collision box size=0.02005 0.099 0.023; visual mesh filename=realsense2_description/meshes/d415.stl
Joints:
- added joint camera_link_joint: type fixed, parent camera_base_link, child camera_link, origin xyz=0 0.02 0.0115 rpy=0 0 0
- added joint realsense_joint: type fixed, parent panda_hand, child camera_base_link, origin xyz=0.035 0 0.036 rpy=0 -1.5707 3.1415
